Commit message: copia launchers (nav2 localization no carga mapa)

File: description/robot_core.xacro (robot description, xacro)
@@ -21,5 +21,5 @@
     </link>
     <!-- BASE_FOOTPRINT LINK -->
-    <!-- <joint name="base_footprint_joint" type="fixed">
+    <joint name="base_footprint_joint" type="fixed">
         <parent link="base_link"/>
         <child link="base_footprint"/>
@@ -27,5 +27,5 @@
     </joint>
     <link name="base_footprint">
-    </link> -->
+    </link>
     <!-- CHASSIS LINK -->
     <joint name="chassis_joint" type="fixed">
